File: 592-kicad-pcb/motherboard/chip_support_misc.kicad_sch (KiCad schematic)
At the start: 7 parts, among them J5 2.54mm jumper, SW1 C318884, U3 SN74LVC1G14DBV, U4 74LVC1T45GW

Commit message: updates to routing
Parts:
- renumbered J5 to J8, R20 to R21, R21 to R22, U3 to U4, U4 to U5
Changed lines of the file:
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@@
 		(on_board yes)
 		(dnp no)
-		(property "Reference" "U3"
+		(property "Reference" "U4"
 			(at 69.596 88.9 0)
 			(effects
@@
 			(project "motherboard"
 				(path "/5b0c97ac-fa03-4db8-b41b-0eee32b6f55d/f049e4ad-bebe-4338-850a-2727de737ae9/43b528c2-ed3f-4c4d-855d-1f88d0a4fadb"
-					(reference "U3")
+					(reference "U4")
 					(unit 1)
 				)
@@
 		(dnp no)
 		(fields_autoplaced yes)
-		(property "Reference" "#PWR057"
+		(property "Reference" "#PWR059"
 			(at 90.17 101.6 0)
 			(effects
@@
 			(project "motherboard"
 				(path "/5b0c97ac-fa03-4db8-b41b-0eee32b6f55d/f049e4ad-bebe-4338-850a-2727de737ae9/43b528c2-ed3f-4c4d-855d-1f88d0a4fadb"
-					(reference "#PWR057")
+					(reference "#PWR059")
 					(unit 1)
 				)
@@
 		(dnp yes)
 		(fields_autoplaced yes)
-		(property "Reference" "J5"
+		(property "Reference" "J8"
 			(at 171.45 81.2799 0)
 			(effects
@@
 			(project "motherboard"
 				(path "/5b0c97ac-fa03-4db8-b41b-0eee32b6f55d/f049e4ad-bebe-4338-850a-2727de737ae9/43b528c2-ed3f-4c4d-855d-1f88d0a4fadb"
-					(reference "J5")
+					(reference "J8")
 					(unit 1)
 				)
@@
 		(dnp no)
 		(fields_autoplaced yes)
-		(property "Reference" "#PWR055"
+		(property "Reference" "#PWR057"
 			(at 43.18 107.95 0)
 			(effects
@@
 			(project "motherboard"
 				(path "/5b0c97ac-fa03-4db8-b41b-0eee32b6f55d/f049e4ad-bebe-4338-850a-2727de737ae9/43b528c2-ed3f-4c4d-855d-1f88d0a4fadb"
-					(reference "#PWR055")
+					(reference "#PWR057")
 					(unit 1)
 				)
@@
 		(dnp no)
 		(fields_autoplaced yes)
-		(property "Reference" "#PWR059"
+		(property "Reference" "#PWR061"
 			(at 144.78 101.6 0)
 			(effects
@@
 			(project "motherboard"
 				(path "/5b0c97ac-fa03-4db8-b41b-0eee32b6f55d/f049e4ad-bebe-4338-850a-2727de737ae9/43b528c2-ed3f-4c4d-855d-1f88d0a4fadb"
-					(reference "#PWR059")
+					(reference "#PWR061")
 					(unit 1)
 				)
@@
 		(on_board yes)
 		(dnp no)
-		(property "Reference" "#PWR058"
+		(property "Reference" "#PWR060"
 			(at 102.87 81.28 0)
 			(effects
@@
 			(project "motherboard"
 				(path "/5b0c97ac-fa03-4db8-b41b-0eee32b6f55d/f049e4ad-bebe-4338-850a-2727de737ae9/43b528c2-ed3f-4c4d-855d-1f88d0a4fadb"
-					(reference "#PWR058")
+					(reference "#PWR060")
 					(unit 1)
 				)
@@
 		(dnp no)
 		(fields_autoplaced yes)
-		(property "Reference" "R20"
+		(property "Reference" "R21"
 			(at 45.72 77.4699 0)
 			(effects
@@
 			(project "motherboard"
 				(path "/5b0c97ac-fa03-4db8-b41b-0eee32b6f55d/f049e4ad-bebe-4338-850a-2727de737ae9/43b528c2-ed3f-4c4d-855d-1f88d0a4fadb"
-					(reference "R20")
+					(reference "R21")
 					(unit 1)
 				)
@@
 		(on_board yes)
 		(dnp no)
-		(property "Reference" "U4"
+		(property "Reference" "U5"
 			(at 89.916 72.644 0)
 			(effects
@@
 			(project "motherboard"
 				(path "/5b0c97ac-fa03-4db8-b41b-0eee32b6f55d/f049e4ad-bebe-4338-850a-2727de737ae9/43b528c2-ed3f-4c4d-855d-1f88d0a4fadb"
-					(reference "U4")
+					(reference "U5")
 					(unit 1)
 				)
@@
 		(on_board yes)
 		(dnp no)
-		(property "Reference" "#PWR056"
+		(property "Reference" "#PWR058"
 			(at 77.47 81.28 0)
 			(effects
@@
 			(project "motherboard"
 				(path "/5b0c97ac-fa03-4db8-b41b-0eee32b6f55d/f049e4ad-bebe-4338-850a-2727de737ae9/43b528c2-ed3f-4c4d-855d-1f88d0a4fadb"
-					(reference "#PWR056")
+					(reference "#PWR058")
 					(unit 1)
 				)
@@
 		(dnp no)
 		(fields_autoplaced yes)
-		(property "Reference" "R21"
+		(property "Reference" "R22"
 			(at 147.32 87.6299 0)
 			(effects
@@
 			(project "motherboard"
 				(path "/5b0c97ac-fa03-4db8-b41b-0eee32b6f55d/f049e4ad-bebe-4338-850a-2727de737ae9/43b528c2-ed3f-4c4d-855d-1f88d0a4fadb"
-					(reference "R21")
+					(reference "R22")
 					(unit 1)
 				)
@@
 		(on_board yes)
 		(dnp no)
-		(property "Reference" "#PWR054"
+		(property "Reference" "#PWR056"
 			(at 43.18 73.66 0)
 			(effects
@@
 			(project "motherboard"
 				(path "/5b0c97ac-fa03-4db8-b41b-0eee32b6f55d/f049e4ad-bebe-4338-850a-2727de737ae9/43b528c2-ed3f-4c4d-855d-1f88d0a4fadb"
-					(reference "#PWR054")
+					(reference "#PWR056")
 					(unit 1)
 				)
